Commit message: Actualizacion 1

File: URDF/robot.urdf (robot description, URDF)
Before this commit: robot robot_inicial, 5 links, 0 joints
Joints:
- added joint 1_joint: type revolute, parent 0_link, child 1_link, origin xyz=0.0 0.0 0.0 rpy=0.0 0.0 0.0, axis 0.0 0.0 1.0, limit lower=-3.14 upper=3.14 effort=1.0 velocity=10.0

Commit message: Actualización rápida

File: URDF/robot.urdf (robot description, URDF)
Before this commit: robot robot_inicial, 5 links, 1 joints
Joints:
- added joint 2_joint: type revolute, parent 1_link, child 2_link, origin xyz=0.5 0.0 0.0 rpy=0.0 0.0 0.0, axis 0.0 0.0 1.0, limit lower=-3.14 upper=3.14 effort=1.0 velocity=10.0

Commit message: Actualización rápida

File: URDF/robot.urdf (robot description, URDF)
Before this commit: robot robot_inicial, 5 links, 2 joints
Joints:
- added joint 3_joint: type revolute, parent 2_link, child 3_link, origin xyz=0.5 0.0 0.0 rpy=0.0 0.0 0.0, axis 0.0 0.0 1.0, limit lower=-3.14 upper=3.14 effort=1.0 velocity=10.0
- added joint p_joint: type fixed, parent 3_link, child p_link, origin xyz=0.5 0.0 0.0 rpy=0.0 0.0 0.0, axis 0.0 0.0 1.0, limit lower=-3.14 upper=3.14 effort=1.0 velocity=10.0

Commit message: Actualización rápida

File: URDF/robot.urdf (robot description, URDF)
Before this commit: robot robot_inicial, 5 links, 4 joints
Links:
- link 1_link: geometry visual box size=0.5 0.05 0.05
- link 2_link: geometry visual box size=0.5 0.05 0.05
- link 3_link: geometry visual box size=0.5 0.05 0.05
- link p_link: geometry visual box size=0.05 0.05 0.05
Joints:
- joint p_joint: axis 0.0 0.0 1.0 -> (none); limit lower=-3.14 upper=3.14 effort=1.0 velocity=10.0 -> (none)

Commit message: Actualización rápida

File: URDF/robot.urdf (robot description, URDF)
Before this commit: robot robot_inicial, 5 links, 4 joints
Links:
- link 1_link: geometry visual box size=0.5 0.05 0.05; visual sphere radius=0.035

Commit message: Actualización rápida

File: URDF/robot.urdf (robot description, URDF)
Before this commit: robot robot_inicial, 5 links, 4 joints
Joints:
- joint 1_joint: origin xyz=0.0 0.0 0.0 rpy=0.0 0.0 0.0 -> xyz=0.0 0.0 0.0 rpy=1.57 0.0 0.0
